File: synth/hardware/Mentor.brd (EAGLE design)
At the start: 200 x 120 mm, 36 parts, among them IC1 MCP23017SO

Commit message: Update - tests and wavefolding
Parts:
- U$3: value (none) -> AUDIO SHIELD
Changed lines of the file:
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@@
 <?xml version="1.0" encoding="utf-8"?>
 <!DOCTYPE eagle SYSTEM "eagle.dtd">
-<eagle version="6.1">
+<eagle version="8.2.1">
 <drawing>
 <settings>
@@
 </class>
 </classes>
-<designrules>
+<designrules name="default">
 <description language="de">&lt;b&gt;EAGLE Design Rules&lt;/b&gt;
 &lt;p&gt;
@@
 <pass name="Default">
 <param name="RoutingGrid" value="50mil"/>
+<param name="AutoGrid" value="1"/>
+<param name="Efforts" value="0"/>
+<param name="TopRouterVariant" value="1"/>
 <param name="tpViaShape" value="round"/>
 <param name="PrefDir.1" value="|"/>
@@
 <element name="CTRL4" library="SparkFun-Switches" package="ENCODER_NOSW" value="ENCODER_NOSW" x="88.9" y="15.24"/>
 <element name="D1" library="SparkFun-LED" package="LED_3MM" value="" x="21.59" y="68.58" smashed="yes" rot="R180">
+<attribute name="NAME" x="21.59" y="67.564" size="0.6096" layer="25" font="vector" ratio="20" rot="R180"/>
 <attribute name="PROD_ID" value="DIO-08794" x="21.59" y="68.58" size="1.778" layer="27" rot="R180" display="off"/>
-<attribute name="NAME" x="21.59" y="67.564" size="0.6096" layer="25" font="vector" ratio="20" rot="R180"/>
 <attribute name="VALUE" x="21.59" y="70.866" size="0.6096" layer="27" font="vector" ratio="20" rot="R180"/>
 </element>
@@
 </element>
 <element name="D2" library="SparkFun-LED" package="LED_3MM" value="" x="21.59" y="60.96" smashed="yes" rot="R180">
+<attribute name="NAME" x="21.59" y="59.944" size="0.6096" layer="25" font="vector" ratio="20" rot="R180"/>
 <attribute name="PROD_ID" value="DIO-08794" x="21.59" y="60.96" size="1.778" layer="27" rot="R180" display="off"/>
-<attribute name="NAME" x="21.59" y="59.944" size="0.6096" layer="25" font="vector" ratio="20" rot="R180"/>
 <attribute name="VALUE" x="21.59" y="63.246" size="0.6096" layer="27" font="vector" ratio="20" rot="R180"/>
 </element>
 <element name="D3" library="SparkFun-LED" package="LED_3MM" value="" x="21.59" y="53.34" smashed="yes" rot="R180">
+<attribute name="NAME" x="21.59" y="52.324" size="0.6096" layer="25" font="vector" ratio="20" rot="R180"/>
 <attribute name="PROD_ID" value="DIO-08794" x="21.59" y="53.34" size="1.778" layer="27" rot="R180" display="off"/>
-<attribute name="NAME" x="21.59" y="52.324" size="0.6096" layer="25" font="vector" ratio="20" rot="R180"/>
 <attribute name="VALUE" x="21.59" y="55.626" size="0.6096" layer="27" font="vector" ratio="20" rot="R180"/>
 </element>
 <element name="D4" library="SparkFun-LED" package="LED_3MM" value="" x="21.59" y="45.72" smashed="yes" rot="R180">
+<attribute name="NAME" x="21.59" y="44.704" size="0.6096" layer="25" font="vector" ratio="20" rot="R180"/>
 <attribute name="PROD_ID" value="DIO-08794" x="21.59" y="45.72" size="1.778" layer="27" rot="R180" display="off"/>
-<attribute name="NAME" x="21.59" y="44.704" size="0.6096" layer="25" font="vector" ratio="20" rot="R180"/>
 <attribute name="VALUE" x="21.59" y="48.006" size="0.6096" layer="27" font="vector" ratio="20" rot="R180"/>
 </element>
 <element name="D5" library="SparkFun-LED" package="LED_3MM" value="" x="21.59" y="38.1" smashed="yes" rot="R180">
+<attribute name="NAME" x="21.59" y="37.084" size="0.6096" layer="25" font="vector" ratio="20" rot="R180"/>
 <attribute name="PROD_ID" value="DIO-08794" x="21.59" y="38.1" size="1.778" layer="27" rot="R180" display="off"/>
-<attribute name="NAME" x="21.59" y="37.084" size="0.6096" layer="25" font="vector" ratio="20" rot="R180"/>
 <attribute name="VALUE" x="21.59" y="40.386" size="0.6096" layer="27" font="vector" ratio="20" rot="R180"/>
 </element>
 <element name="D6" library="SparkFun-LED" package="LED_3MM" value="" x="21.59" y="30.48" smashed="yes" rot="R180">
+<attribute name="NAME" x="21.59" y="29.464" size="0.6096" layer="25" font="vector" ratio="20" rot="R180"/>
 <attribute name="PROD_ID" value="DIO-08794" x="21.59" y="30.48" size="1.778" layer="27" rot="R180" display="off"/>
-<attribute name="NAME" x="21.59" y="29.464" size="0.6096" layer="25" font="vector" ratio="20" rot="R180"/>
 <attribute name="VALUE" x="21.59" y="32.766" size="0.6096" layer="27" font="vector" ratio="20" rot="R180"/>
 </element>
 <element name="D7" library="SparkFun-LED" package="LED_3MM" value="" x="56.8325" y="45.72" smashed="yes" rot="R180">
+<attribute name="NAME" x="56.8325" y="44.704" size="0.6096" layer="25" font="vector" ratio="20" rot="R180"/>
 <attribute name="PROD_ID" value="DIO-08794" x="56.8325" y="45.72" size="1.778" layer="27" rot="R180" display="off"/>
-<attribute name="NAME" x="56.8325" y="44.704" size="0.6096" layer="25" font="vector" ratio="20" rot="R180"/>
 <attribute name="VALUE" x="56.8325" y="48.006" size="0.6096" layer="27" font="vector" ratio="20" rot="R180"/>
 </element>
@@
 </element>
 <element name="LCD" library="SparkFun-Connectors" package="1X04_LONGPADS" value="" x="191.77" y="57.15" smashed="yes" rot="R270">
+<attribute name="NAME" x="186.182" y="57.15" size="2.1844" layer="25" font="vector" rot="R270"/>
 <attribute name="PROD_ID" value="CONN-09696" x="191.77" y="57.15" size="1.778" layer="27" rot="R270" display="off"/>
-<attribute name="NAME" x="186.182" y="57.15" size="2.1844" layer="25" font="vector" rot="R270"/>
 <attribute name="VALUE" x="189.103" y="58.42" size="0.6096" layer="27" font="vector" ratio="20" rot="R270"/>
 </element>
 <element name="LINE_OUT" library="SparkFun-Connectors" package="AUDIO-JACK" value="" x="184.15" y="115.57" smashed="yes" rot="R270">
+<attribute name="PROD_ID" value="CONN-08774" x="184.15" y="115.57" size="1.778" layer="27" rot="R270" display="off"/>
 <attribute name="SF_ID" value="PRT-08032" x="184.15" y="115.57" size="1.778" layer="27" rot="R270" display="off"/>
-<attribute name="PROD_ID" value="CONN-08774" x="184.15" y="115.57" size="1.778" layer="27" rot="R270" display="off"/>
 <attribute name="VALUE" x="181.483" y="116.84" size="0.6096" layer="27" font="vector" ratio="20" rot="R270"/>
 </element>
@@
 <element name="SEL" library="SparkFun-Switches" package="ENCODER_NOSW" value="ENCODER_NOSW" x="15.24" y="15.24"/>
 <element name="U$2" library="Teensy4.0_SIMPLE" package="TEENSY4.0_SIMPLE" value="TEENSY4.0_SIMPLE" x="123.19" y="102.87" smashed="yes"/>
-<element name="U$3" library="Teensy_Audioshield_alt" package="AUDIOSHIELD" value="" x="153.67" y="101.6" smashed="yes" rot="R270"/>
+<element name="U$3" library="Teensy_Audioshield_alt" package="AUDIOSHIELD" value="AUDIO SHIELD" x="153.67" y="101.6" smashed="yes" rot="R270"/>
 <element name="VOL_PWR" library="alps_japan_potentiometers" package="RK097-SINGLE-W/SWITCH" value="10K" x="16.51" y="115.57" rot="R180"/>
 <element name="R8" library="resistor" package="R0603" value="500" x="15.24" y="68.58" rot="MR0"/>
@@
 </element>
 <element name="OK1" library="optocoupler" package="DIL6-SMD" value="H11L1MS" x="16.51" y="88.9" rot="MR180">
+<attribute name="MF" value="" x="16.51" y="88.9" size="1.778" layer="28" rot="MR180" display="off"/>
 <attribute name="MPN" value="" x="16.51" y="88.9" size="1.778" layer="28" rot="MR180" display="off"/>
-<attribute name="MF" value="" x="16.51" y="88.9" size="1.778" layer="28" rot="MR180" display="off"/>
 <attribute name="OC_FARNELL" value="unknown" x="16.51" y="88.9" size="1.778" layer="28" rot="MR180" display="off"/>
 <attribute name="OC_NEWARK" value="unknown" x="16.51" y="88.9" size="1.778" layer="28" rot="MR180" display="off"/>
@@
 <signal name="VCC">
 <contactref element="VOL_PWR" pad="P2"/>
-<contactref element="U$2" pad="3.3V@1" route="any"/>
+<contactref element="U$2" pad="3.3V@1" route="any" routetag="G$1.3.3V"/>
 <contactref element="R3" pad="2"/>
 <contactref element="U$3" pad="3V"/>
